Commit message: Adjust the z of the TCP

File: project_praktikum/robot_description/urdf/robotron.urdf (robot description, URDF)
Before this commit: robot robotron, 9 links, 8 joints
Joints:
- joint tool_link__eff: origin xyz=0.000 0.000 -0.188 rpy=0 0 -1.57 -> xyz=0.000 0.000 -0.141 rpy=0 0 -1.57

Commit message: mechanical compensation solved and first frasing attempt

File: project_praktikum/robot_description/urdf/robotron.urdf (robot description, URDF)
Before this commit: robot robotron, 9 links, 8 joints
Joints:
- joint tool_link__eff: origin xyz=0.000 0.000 -0.141 rpy=0 0 -1.57 -> xyz=0.002 -0.002 -0.141 rpy=0 0 -1.57
