Commit message: dold_gui_6 update

File: 6-dof-arm-pick-and-place/urdf/urdf_arm.urdf (robot description, URDF)
Before this commit: robot manipulator, 9 links, 8 joints
Links:
- added link link7, mass 0.1; collision box size=0.02 0.02 0.15; visual box size=0.02 0.02 0.15
- link tcp: geometry collision box size=0 0 0; visual box size=0 0 0
Joints:
- removed joint joint6_tcp
- added joint joint7: type revolute, parent link6, child link7, origin xyz=0 0 0.3 rpy=0 0 0, axis 0 0 1, limit lower=-3.14 upper=3.14 effort=100 velocity=1
- added joint joint7_tcp: type fixed, parent link7, child tcp, origin xyz=0 0 0 rpy=0 0 0

Commit message: updated urdf joints measurements

File: 6-dof-arm-pick-and-place/urdf/urdf_arm.urdf (robot description, URDF)
Before this commit: robot manipulator, 10 links, 9 joints
Joints:
- joint joint2: limit lower=-1.72 upper=1.72 effort=100 velocity=1 -> lower=-1.4835 upper=1.4835 effort=100 velocity=1
- joint joint3: limit lower=-1.72 upper=1.72 effort=100 velocity=1 -> lower=-1.4835 upper=1.4835 effort=100 velocity=1; origin xyz=0 0 0.32 rpy=0 0 0 -> xyz=0 0 0.33 rpy=0 0 0
- joint joint4: limit lower=-1.72 upper=1.72 effort=100 velocity=1 -> lower=-1.4835 upper=1.4835 effort=100 velocity=1; origin xyz=0 0 0.32 rpy=0 0 0 -> xyz=0 0 0.33 rpy=0 0 0
- joint joint6: limit lower=-1.72 upper=1.72 effort=100 velocity=1 -> lower=-1.4835 upper=1.4835 effort=100 velocity=1; origin xyz=0 0 0.2 rpy=0 0 0 -> xyz=0 0 0.23 rpy=0 0 0
- joint joint7: origin xyz=0 0 0.3 rpy=0 0 0 -> xyz=0 0 0.263 rpy=0 0 0

Commit message: changed gcode generation format

File: 6-dof-arm-pick-and-place/urdf/urdf_arm.urdf (robot description, URDF)
Before this commit: robot manipulator, 10 links, 9 joints
Joints:
- joint joint3: origin xyz=0 0 0.33 rpy=0 0 0 -> xyz=0 0 0.32 rpy=0 0 0
- joint joint4: origin xyz=0 0 0.33 rpy=0 0 0 -> xyz=0 0 0.32 rpy=0 0 0
- joint joint7: origin xyz=0 0 0.263 rpy=0 0 0 -> xyz=0 0 0.264 rpy=0 0 0

Commit message: z joint negativ constraint

File: 6-dof-arm-pick-and-place/urdf/urdf_arm.urdf (robot description, URDF)
Before this commit: robot manipulator, 10 links, 9 joints
Joints:
- joint joint3: limit lower=-1.4835 upper=1.4835 effort=100 velocity=1 -> lower=-1.4835 upper=0.15 effort=100 velocity=1

Commit message: joint 1 constraint to 200 deg

File: 6-dof-arm-pick-and-place/urdf/urdf_arm.urdf (robot description, URDF)
Before this commit: robot manipulator, 10 links, 9 joints
Joints:
- joint joint1: limit lower=-6.28 upper=6.28 effort=100 velocity=1 -> lower=-3.5 upper=3.5 effort=100 velocity=1
